File: Hardware/flight_comp.kicad_sch (KiCad schematic)
At the start: 34 parts, among them J2 ARM_SWD_TC2030, J4 USB_C_Receptacle_USB2.0_16P, U1 STM32F405RGTx, U4 W25Q32JVSS, U5 24LC64, U8 USBLC6-2SC6, Y1 8mHz, Y2 32.768 kHz

Commit message: PCB added, minor changes
Parts:
- added BZ1: Buzzer, Buzzer_Beeper:Buzzer_CUI_CPT-9019S-SMT, symbol Device:Buzzer
- added Q5: PMBT2222A, Package_TO_SOT_SMD:SOT-23, symbol Transistor_BJT:PMBT2222A
- added R33: 1k, Resistor_SMD:R_0603_1608Metric, symbol Device:R
- added SW1: NRST, Button_Switch_SMD:SW_SPST_CK_RS282G05A3, symbol Switch:SW_Push
- added SW2: BOOT0, Button_Switch_SMD:SW_SPST_CK_RS282G05A3, symbol Switch:SW_Push
- BT1: footprint Battery:BatteryHolder_Keystone_500 -> Battery:BatteryHolder_Keystone_2998_1x6.8mm
- C10, C11: value C -> 0.1uF; footprint (none) -> Capacitor_SMD:C_0603_1608Metric
- C20, C23, C27, C28, C29, C30, C31, C32, C33, C6, C7, C8, C9: footprint (none) -> Capacitor_SMD:C_0603_1608Metric
- L2: footprint (none) -> Inductor_SMD:L_0603_1608Metric
- R21, R28, R29, R32, R5, R6, R7: footprint (none) -> Resistor_SMD:R_0603_1608Metric
Connections:
- net +3.3V: now also R5.2, SW2.1; no longer R5.1
- net GND: now also Q5.2 (E), SW1.1
- net BUZZ: now reaches U1.11 (PC3)
- net BUZZ: now also R33.1
- net at R6.2, U1.60 (BOOT0): now also SW2.2
- net at U1.7 (NRST): now also R5.1, SW1.2; no longer R5.2
- new net: Q5.1 (B), R33.2
- new net: BZ1.2 (-), Q5.3 (C)
- new net VCC: BZ1.1 (+)
Other:
- moved on the sheet: C10, C33, R5, R6
