File: Hardware/flight_comp.kicad_sch (KiCad schematic)
At the start: 43 parts, among them J2 ARM_SWD_TC2030, J4 USB_C_Receptacle_USB2.0_16P, Q5 PMBT2222A, SW1 NRST, SW2 BOOT0, U1 STM32F405RGTx, U4 W25Q32JVSS, U5 24LC64, U8 USBLC6-2SC6, Y1 8mHz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

Commit message: camera, impedance control
Parts:
- removed J2: ARM_SWD_TC2030, Connector:Tag-Connect_TC2030-IDC-NL_2x03_P1.27mm_Vertical, symbol Connector:Conn_ARM_SWD_TagConnect_TC2030-NL
- added J2: TC2030, Connector:Tag-Connect_TC2030-IDC-NL_2x03_P1.27mm_Vertical, symbol Connector:TC2030
- C20, C23: footprint Capacitor_SMD:C_0603_1608Metric -> Capacitor_SMD:C_0402_1005Metric
Connections:
- net +3.3V: now also J2.1
- net GND: now also J2.6
- net SYS_SWCLK: now also J2.4
- net SYS_SWDIO: now also J2.3
- net SYS_SWO: now also J2.2
- net CAMERA_SWITCH: now reaches U1.8 (PC0)
- no-connect marks 8 -> 7
Changed lines of the file:
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@@
 	)
 	(no_connect
-		(at 256.54 76.2)
+		(at 233.68 83.82)
 	)
 	(no_connect
@@
 	)
 	(no_connect
-		(at 148.59 53.34)
-	)
-	(no_connect
 		(at 148.59 55.88)
 	)
@@
 	(wire
 		(pts
+			(xy 232.41 78.74) (xy 233.68 78.74)
+		)
+		(stroke
+			(width 0)
+			(type default)
+		)
+	)
+	(wire
+		(pts
 			(xy 67.31 91.44) (xy 69.85 91.44)
 		)
@@
 	(wire
 		(pts
+			(xy 247.65 83.82) (xy 246.38 83.82)
+		)
+		(stroke
+			(width 0)
+			(type default)
+		)
+	)
+	(wire
+		(pts
 			(xy 140.97 99.06) (xy 148.59 99.06)
 		)
@@
 	(global_label "SYS_SWDIO"
 		(shape input)
-		(at 256.54 83.82 0)
+		(at 233.68 81.28 180)
 		(fields_autoplaced yes)
 		(effects
@@
 				(size 1.27 1.27)
 			)
-			(justify left)
+			(justify right)
 		)
 		(property "Intersheetrefs" "${INTERSHEET_REFS}"
-			(at 269.8666 83.82 0)
+			(at 220.3534 81.28 0)
 			(effects
 				(font
 					(size 1.27 1.27)
 				)
-				(justify left)
+				(justify right)
 				(hide yes)
 			)
@@
 		)
 	)
+	(global_label "CAMERA_SWITCH"
+		(shape output)
+		(at 148.59 53.34 180)
+		(fields_autoplaced yes)
+		(effects
+			(font
+				(size 1.27 1.27)
+			)
+			(justify right)
+		)
+		(property "Intersheetrefs" "${INTERSHEET_REFS}"
+			(at 130.4858 53.34 0)
+			(effects
+				(font
+					(size 1.27 1.27)
+				)
+				(justify right)
+				(hide yes)
+			)
+		)
+	)
 	(global_label "LORA_SCK"
 		(shape input)
@@
 	(global_label "SYS_SWCLK"
 		(shape input)
-		(at 256.54 81.28 0)
+		(at 246.38 81.28 0)
 		(fields_autoplaced yes)
 		(effects
@@
 		)
 		(property "Intersheetrefs" "${INTERSHEET_REFS}"
-			(at 270.2294 81.28 0)
+			(at 260.0694 81.28 0)
 			(effects
 				(font
@@
 	(global_label "SYS_SWO"
 		(shape input)
-		(at 256.54 86.36 0)
+		(at 246.38 78.74 0)
 		(fields_autoplaced yes)
 		(effects
@@
 		)
 		(property "Intersheetrefs" "${INTERSHEET_REFS}"
-			(at 267.9918 86.36 0)
+			(at 257.8318 78.74 0)
 			(effects
 				(font
@@
 			)
 		)
-		(property "Footprint" "Capacitor_SMD:C_0603_1608Metric"
+		(property "Footprint" "Capacitor_SMD:C_0402_1005Metric"
 			(at 28.9052 101.6 0)
 			(effects
@@
 	)
 	(symbol
-		(lib_id "Connector:Conn_ARM_SWD_TagConnect_TC2030-NL")
-		(at 248.92 81.28 0)
-		(unit 1)
-		(exclude_from_sim no)
-		(in_bom no)
-		(on_board yes)
-		(dnp no)
-		(fields_autoplaced yes)
-		(property "Reference" "J2"
-			(at 242.57 80.0099 0)
-			(effects
-				(font
-					(size 1.27 1.27)
-				)
-				(justify right)
-			)
-		)
-		(property "Value" "ARM_SWD_TC2030"
-			(at 242.57 82.5499 0)
-			(effects
-				(font
-					(size 1.27 1.27)
-				)
-				(justify right)
-			)
-		)
-		(property "Footprint" "Connector:Tag-Connect_TC2030-IDC-NL_2x03_P1.27mm_Vertical"
-			(at 248.92 99.06 0)
-			(effects
-				(font
-					(size 1.27 1.27)
-				)
-				(hide yes)
-			)
-		)
-		(property "Datasheet" "https://www.tag-connect.com/wp-content/uploads/bsk-pdf-manager/TC2030-CTX_1.pdf"
-			(at 248.92 96.52 0)
-			(effects
-				(font
-					(size 1.27 1.27)
-				)
-				(hide yes)
-			)
-		)
-		(property "Description" "Tag-Connect ARM Cortex SWD JTAG connector, 6 pin, no legs"
-			(at 248.92 81.28 0)
-			(effects
-				(font
-					(size 1.27 1.27)
-				)
-				(hide yes)
-			)
-		)
-		(pin "3"
-		)
-		(pin "2"
-		)
-		(pin "5"
-		)
-		(pin "4"
-		)
-		(pin "1"
-		)
-		(pin "6"
-		)
-		(instances
-			(project ""
-				(path "/99100214-bcab-4638-96e7-2342f837a8e5"
-					(reference "J2")
-					(unit 1)
-				)
-			)
-		)
-	)
-	(symbol
 		(lib_id "Device:R")
 		(at 31.75 52.07 0)
@@
 	(symbol
 		(lib_id "power:GND")
-		(at 246.38 91.44 0)
+		(at 247.65 83.82 0)
 		(unit 1)
 		(exclude_from_sim no)
@@
 		(fields_autoplaced yes)
 		(property "Reference" "#PWR035"
-			(at 246.38 97.79 0)
+			(at 247.65 90.17 0)
 			(effects
 				(font
@@
 		)
 		(property "Value" "GND"
-			(at 246.38 96.52 0)
+			(at 247.65 88.9 0)
 			(effects
 				(font
@@
 		)
 		(property "Footprint" ""
-			(at 246.38 91.44 0)
+			(at 247.65 83.82 0)
 			(effects
 				(font
@@
 		)
 		(property "Datasheet" ""
-			(at 246.38 91.44 0)
+			(at 247.65 83.82 0)
 			(effects
 				(font
@@
 		)
 		(property "Description" "Power symbol creates a global label with name \"GND\" , ground"
-			(at 246.38 91.44 0)
+			(at 247.65 83.82 0)
 			(effects
 				(font
@@
 			)
 		)
-		(property "Footprint" "Capacitor_SMD:C_0603_1608Metric"
+		(property "Footprint" "Capacitor_SMD:C_0402_1005Metric"
 			(at 41.6052 101.6 0)
 			(effects
@@
 	)
 	(symbol
+		(lib_id "Connector:TC2030")
+		(at 238.76 81.28 0)
+		(unit 1)
+		(exclude_from_sim no)
+		(in_bom no)
+		(on_board yes)
+		(dnp no)
+		(fields_autoplaced yes)
+		(property "Reference" "J2"
+			(at 240.03 68.58 0)
+			(effects
+				(font
+					(size 1.27 1.27)
+				)
+			)
+		)
+		(property "Value" "TC2030"
+			(at 240.03 71.12 0)
+			(effects
+				(font
+					(size 1.27 1.27)
+				)
+			)
+		)
+		(property "Footprint" "Connector:Tag-Connect_TC2030-IDC-NL_2x03_P1.27mm_Vertical"
+			(at 240.03 81.28 0)
+			(effects
+				(font
+					(size 1.27 1.27)
+				)
+				(hide yes)
+			)
+		)
+		(property "Datasheet" "https://www.tag-connect.com/wp-content/uploads/bsk-pdf-manager/2019/12/TC2030-IDC-NL-Datasheet-Rev-B.pdf"
+			(at 240.03 81.28 0)
+			(effects
+				(font
+					(size 1.27 1.27)
+				)
+				(hide yes)
+			)
+		)
+		(property "Description" "Tag-Connect’s 6-pins connector"
+			(at 238.76 81.28 0)
+			(effects
+				(font
+					(size 1.27 1.27)
+				)
+				(hide yes)
+			)
+		)
+		(pin "1"
+		)
+		(pin "6"
+		)
+		(pin "3"
+		)
+		(pin "4"
+		)
+		(pin "2"
+		)
+		(pin "5"
+		)
+		(instances
+			(project ""
+				(path "/99100214-bcab-4638-96e7-2342f837a8e5"
+					(reference "J2")
+					(unit 1)
+				)
+			)
+		)
+	)
+	(symbol
 		(lib_id "power:GND")
 		(at 270.51 121.92 0)
@@
 	(symbol
 		(lib_id "power:+3.3V")
-		(at 246.38 71.12 0)
+		(at 232.41 78.74 0)
 		(unit 1)
 		(exclude_from_sim no)
@@
 		(fields_autoplaced yes)
 		(property "Reference" "#PWR034"
-			(at 246.38 74.93 0)
+			(at 232.41 82.55 0)
 			(effects
 				(font
@@
 		)
 		(property "Value" "+3.3V"
-			(at 246.38 66.04 0)
+			(at 232.41 73.66 0)
 			(effects
 				(font
@@
 		)
 		(property "Footprint" ""
-			(at 246.38 71.12 0)
+			(at 232.41 78.74 0)
 			(effects
 				(font
@@
 		)
 		(property "Datasheet" ""
-			(at 246.38 71.12 0)
+			(at 232.41 78.74 0)
 			(effects
 				(font
@@
 		)
 		(property "Description" "Power symbol creates a global label with name \"+3.3V\""
-			(at 246.38 71.12 0)
+			(at 232.41 78.74 0)
 			(effects
 				(font
