File: Hardware/power.kicad_sch (KiCad schematic)
At the start: 52 parts, among them IC4 TPS259531DSGR, J10 CAMERA_CONN_01, J11 CAMERA_CONN_02, J13 CAMERA_CONN_03, J3 XT30, J5 Conn_01x02, J6 Conn_01x02, J7 SERVO_CONN_01, J8 SERVO_CONN_02, J9 SERVO_CONN_02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

Commit message: camera, impedance control
Parts:
- added SW3: EG2219, Button_Switch_SMD:SW_DPDT_CK_JS202011JCQN, symbol Switch:SW_DPDT_x2
- C24: footprint 6TPF470MFH:6TPF470MFH -> Capacitor_Tantalum_SMD:CP_EIA-3216-10_Kemet-I
- F1: footprint Fuse:Fuse_0805_2012Metric -> Fuse:Fuse_1206_3216Metric
- IC4: footprint SON50P200X200X80-9N -> Package_SON:WSON-8-1EP_2x2mm_P0.5mm_EP0.9x1.6mm_ThermalVias
- J10, J11, J13: footprint TerminalBlock_4Ucon:TerminalBlock_4Ucon_1x02_P3.50mm_Vertical -> TerminalBlock:TerminalBlock_Xinya_XY308-2.54-2P_1x02_P2.54mm_Horizontal
Connections:
- net GND: now also SW3.1 (A), SW3.4 (A)
- net PYRO_1: now also SW3.3 (C); no longer U11.3 (IN+)
- net PYRO_2: now also SW3.6 (C); no longer U12.3 (IN+)
- net TIM5_CH1: now also R18.1; no longer R19.2
- net TIM5_CH2: now also R19.2; no longer R18.1
- new net: SW3.2 (B), U11.3 (IN+)
- new net: SW3.5 (B), U12.3 (IN+)

Commit message: final touches
Parts:
- added unit 1 of SW3
Connections:
- net GND: now also SW3.1 (A); no longer SW3.1 (A)
- net PYRO_1: now also SW3.3 (C); no longer SW3.3 (C)
- net at U11.3 (IN+): now also SW3.2 (B); no longer SW3.2 (B)
