File: Hardware/flight_comp.kicad_pcb (KiCad board)
At the start: 2 copper layers, 86.8 x 48.2 mm, 109 parts, among them IC1 BMP388, J1 Conn_Coaxial, J12 Conn_Coaxial, J2 ARM_SWD_TC2030, J3 XT30, J4 USB_C_Receptacle_USB2.0_16P, J5 Conn_01x02, J6 Conn_01x02, J7 SERVO_CONN_01, J8 SERVO_CONN_02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

Commit message: PCB silkscreen, PCB dimensions
Parts:
- added H1: MountingHole, MountingHole:MountingHole_3.2mm_M3, F.Cu at (78.0, 126.1)
- added H2: MountingHole, MountingHole:MountingHole_3.2mm_M3, F.Cu at (78.0, 85.3)
- added H3: MountingHole, MountingHole:MountingHole_3.2mm_M3, F.Cu at (157.2, 85.3)
- added H4: MountingHole, MountingHole:MountingHole_3.2mm_M3, F.Cu at (157.2, 126.1)
- BT1: value CR1220 -> MC621
- moved J12 1.71 mm to (156.2, 118.1)
- moved C41 1.70 mm to (134.6, 119.5)
- moved R26 1.70 mm to (150.4, 124.1)
- moved R27 1.70 mm to (150.4, 125.7)
- moved U2 1.70 mm to (142.2, 122.1)
- moved C42 1.70 mm to (134.6, 120.9)
- moved D5 1.70 mm to (149.4, 119.4)
- moved R48 1.70 mm to (135.2, 123.2)
- moved TX4 1.70 mm to (132.4, 123.2)
- moved U11 1.45 mm to (87.6, 91.2)
- moved Q3 1.45 mm to (87.2, 95.3)
- moved R15 1.45 mm to (90.2, 93.3)
- moved J5 1.45 mm to (79.6, 91.8)
- moved J1 0.60 mm to (156.2, 104.6)
- moved R16 0.50 mm to (90.2, 102.4)
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Routing:
- net GPS_TX: track 23.0 -> 21.1 mm
- net GPS_RX: track 20.6 -> 18.9 mm
- net Net-(D5-A2): track 9.72 -> 10.9 mm
- net PYRO_2: track 51.9 -> 50.9 mm
- net PYRO_1: track 53.6 -> 54.3 mm
- net GND: track 6.65 -> 6.93 mm, vias 17 -> 18
Other:
- board size 86.8 x 48.2 mm -> 86.7 x 48.2 mm
- board text added: "+ -"
- board text added: "2-3S Li-Ion >=20A"
- board text added: "BOOT0"
- board text added: "GND VCC S2 S1"
- board text added: "GND VCC S3 S4"
- board text added: "GND VCC S5 S6"
- board text added: "NRST"
- board text added: "PYRO1"
- board text added: "PYRO2"
- board text added: "SWD"
- board text added: "TYPE MC621"

Commit message: Minor changes in silkscreen and power rails
Routing:
- net GND: track 6.93 -> 14.3 mm, vias 18 -> 19
Other:
- board text added: "<"
- board text added: "PG"
- board text added: "STATUS"
- board text added: "X"
- board text added: "Y"
- board text added: "Z"

Commit message: Kaut ko palaboju
Parts:
- moved J12 1.96 mm to (156.2, 116.1)
- moved H1 0.35 mm to (78.2, 125.8)
- moved H2 0.35 mm to (78.2, 85.6)
- moved H3 0.35 mm to (156.9, 85.6)
- moved H4 0.35 mm to (156.9, 125.8)
Changed lines of the file:
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@@
 	(footprint "MountingHole:MountingHole_3.2mm_M3"
 		(layer "F.Cu")
-		(at 77.95 126.1)
+		(at 78.2 125.85)
 		(descr "Mounting Hole 3.2mm, M3, no annular, generated by kicad-footprint-generator mountinghole.py")
 		(tags "mountinghole M3")
@@
 	(footprint "Connector_Coaxial:SMA_Molex_73251-2200_Horizontal"
 		(layer "F.Cu")
-		(at 156.24 118.1 -90)
+		(at 156.24 116.14 -90)
 		(descr "https://tools.molex.com/pdm_docs/sd/732512200_sd.pdf")
 		(tags "SMA THT Female Jack Horizontal")
@@
 	(footprint "MountingHole:MountingHole_3.2mm_M3"
 		(layer "F.Cu")
-		(at 77.95 85.35)
+		(at 78.2 85.6)
 		(descr "Mounting Hole 3.2mm, M3, no annular, generated by kicad-footprint-generator mountinghole.py")
 		(tags "mountinghole M3")
@@
 	(footprint "MountingHole:MountingHole_3.2mm_M3"
 		(layer "F.Cu")
-		(at 157.2 126.1)
+		(at 156.95 125.85)
 		(descr "Mounting Hole 3.2mm, M3, no annular, generated by kicad-footprint-generator mountinghole.py")
 		(tags "mountinghole M3")
@@
 	(footprint "MountingHole:MountingHole_3.2mm_M3"
 		(layer "F.Cu")
-		(at 157.2 85.35)
+		(at 156.95 85.6)
 		(descr "Mounting Hole 3.2mm, M3, no annular, generated by kicad-footprint-generator mountinghole.py")
 		(tags "mountinghole M3")
@@
 	)
 	(segment
-		(start 91.567832 119.1375)
-		(end 91.4 119.1375)
-		(width 1)
-		(layer "F.Cu")
-		(net 1)
-	)
-	(segment
 		(start 107.95 109.35)
 		(end 107.7 109.1)
@@
 	)
 	(segment
-		(start 151.2 118.1)
-		(end 156.38 118.1)
+		(start 153.16 116.14)
+		(end 156.24 116.14)
 		(width 0.2)
 		(layer "B.Cu")
@@
 	)
 	(segment
-		(start 150.6 118.7)
-		(end 151.2 118.1)
-		(width 0.2)
-		(layer "B.Cu")
-		(net 97)
-	)
-	(segment
-		(start 156.38 118.1)
-		(end 155.63 118.85)
+		(start 149.65 118.85)
+		(end 149.4 118.6)
 		(width 0.2)
 		(layer "B.Cu")
@@
 	)
 	(segment
-		(start 149.65 118.85)
-		(end 149.4 118.6)
+		(start 150.6 118.7)
+		(end 153.16 116.14)
 		(width 0.2)
 		(layer "B.Cu")
@@
 		(layers "F.Cu" "B.Cu")
 		(hatch edge 0.5)
-		(connect_pads
+		(connect_pads yes
 			(clearance 0.2)
 		)
@@
 		(polygon
 			(pts
-				(xy 68.95 73.6) (xy 68.95 133.1) (xy 164.45 133.35) (xy 164.2 75.6)
+				(xy 69.2 76.85) (xy 68.95 133.1) (xy 164.45 133.35) (xy 164.7 76.85)
 			)
 		)
