File: Hardware/flight_comp.kicad_pcb (KiCad board)
At the start: 2 copper layers, 86.7 x 48.2 mm, 113 parts, among them IC1 BMP388, J1 Conn_Coaxial, J12 Conn_Coaxial, J2 ARM_SWD_TC2030, J3 XT30, J4 USB_C_Receptacle_USB2.0_16P, J5 Conn_01x02, J6 Conn_01x02, J7 SERVO_CONN_01, J8 SERVO_CONN_02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

Commit message: camera, impedance control
Parts:
- added C18: 10uF, Capacitor_SMD:C_0603_1608Metric, B.Cu at (80.2, 88.6)
- added C19: 22uF, Capacitor_SMD:C_0603_1608Metric, B.Cu at (84.0, 87.6)
- added C21: 0.1uF, Capacitor_SMD:C_0402_1005Metric, F.Cu at (103.1, 123.3)
- added C22: 0.1uF, Capacitor_SMD:C_0402_1005Metric, F.Cu at (103.1, 125.3)
- added C24: 6TPF470MFH, Capacitor_Tantalum_SMD:CP_EIA-3216-10_Kemet-I, F.Cu at (104.8, 127.3)
- added D2: D_TVS, Diode_SMD:D_SOD-523, B.Cu at (149.9, 105.1)
- added IC4: TPS259531DSGR, Package_SON:WSON-8-1EP_2x2mm_P0.5mm_EP0.9x1.6mm_ThermalVias, F.Cu at (104.9, 124.3)
- added J10: CAMERA_CONN_01, TerminalBlock:TerminalBlock_Xinya_XY308-2.54-2P_1x02_P2.54mm_Horizontal, F.Cu at (100.3, 126.0)
- added J11: CAMERA_CONN_02, TerminalBlock:TerminalBlock_Xinya_XY308-2.54-2P_1x02_P2.54mm_Horizontal, F.Cu at (93.6, 126.0)
- added J13: CAMERA_CONN_03, TerminalBlock:TerminalBlock_Xinya_XY308-2.54-2P_1x02_P2.54mm_Horizontal, F.Cu at (86.8, 126.0)
- added R34: 5k, Resistor_SMD:R_0402_1005Metric, F.Cu at (105.6, 128.9)
- added SW3: EG2219, Button_Switch_SMD:SW_DPDT_CK_JS202011JCQN, F.Cu at (88.2, 85.8)
- added U7: AMS1117-5.0, Package_TO_SOT_SMD:SOT-223-3_TabPin2, B.Cu at (86.2, 93.6)
- C20, C23: footprint Capacitor_SMD:C_0603_1608Metric -> Capacitor_SMD:C_0402_1005Metric
- F1: footprint Fuse:Fuse_0805_2012Metric -> Fuse:Fuse_1206_3216Metric
- J2: value ARM_SWD_TC2030 -> TC2030
- moved BZ1 13.8 mm to (142.8, 86.8), turned to 180 degrees
- moved BT1 11.8 mm to (126.7, 86.8)
- moved C14 8.05 mm to (97.3, 119.4)
- moved R31 8.05 mm to (95.5, 119.4)
- moved R18 7.62 mm to (120.2, 89.3), turned to 90 degrees
- moved D6 7.05 mm to (101.2, 120.6), turned to 0 degrees
- moved R30 6.90 mm to (94.6, 116.8), turned to 0 degrees
- moved J7 6.85 mm to (117.6, 88.7)
- moved R19 6.22 mm to (112.6, 89.3), turned to -90 degrees
- moved R33 5.18 mm to (134.8, 93.8)
- moved Q5 4.80 mm to (135.8, 90.2)
- moved R22 4.29 mm to (111.4, 89.3), turned to 90 degrees
- moved J8 3.52 mm to (109.0, 88.7)
- moved R23 2.80 mm to (103.9, 89.3), turned to -90 degrees
- moved C23 1.67 mm to (127.8, 93.2), turned to 0 degrees
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Connections:
- net /BUZZ renamed BUZZ
- net /EEP_SCL renamed EEP_SCL
- net /EEP_SDA renamed EEP_SDA
- net /EEP_WP renamed EEP_WP
- net /FLASH_CS renamed FLASH_CS
- net /FLASH_MISO renamed FLASH_MISO
- net /FLASH_MOSI renamed FLASH_MOSI
- net /FLASH_SCK renamed FLASH_SCK
- net /FLASH_WP renamed FLASH_WP
- net /LED renamed LED
- net /OSC32_IN renamed OSC32_IN
- net /OSC32_OUT renamed OSC32_OUT
- net /OSC_IN renamed OSC_IN
- net /OSC_OUT renamed OSC_OUT
- net /SYS_SWCLK renamed SYS_SWCLK
- net /USB_DN renamed USB_DN
- net /USB_DP renamed USB_DP
- D4 pad 3: +3.3V -> +5V
- J2 pad 2: /SYS_SWDIO -> SYS_SWO
- J2 pad 3: unconnected-(J2-~{RESET}-Pad3) -> SYS_SWDIO
- J2 pad 5: GND -> unconnected-(J2-Pad5)
- J2 pad 6: /SYS_SWO -> GND
- J7 pad 3: VCC -> +5V
- J7 pad 4: VCC -> +5V
- J8 pad 3: VCC -> +5V
- J8 pad 4: VCC -> +5V
- J9 pad 3: VCC -> +5V
- J9 pad 4: VCC -> +5V
- R18 pad 1: TIM5_CH2 -> TIM5_CH1
- R19 pad 2: TIM5_CH1 -> TIM5_CH2
- U1 pad 46: /SYS_SWDIO -> SYS_SWDIO
- U1 pad 55: /SYS_SWO -> SYS_SWO
- U1 pad 8: unconnected-(U1-PC0-Pad8) -> CAMERA_SWITCH
- U11 pad 3: PYRO_1 -> Net-(SW3A-B)
- U12 pad 3: PYRO_2 -> Net-(SW3B-B)
Routing:
- net +5V: track 0.00 -> 74.5 mm, vias 0 -> 2
- net CAMERA_SWITCH: track 0.00 -> 36.0 mm, vias 0 -> 2
- net VCC: track 73.2 -> 40.3 mm, vias 2 -> 4
- net Net-(C24-+): track 0.00 -> 26.4 mm
- net +3.3V: track 233.3 -> 251.7 mm
- net Net-(SW3B-B): track 0.00 -> 17.4 mm, vias 0 -> 2
- net SYS_SWDIO: track 0.00 -> 12.0 mm
- net SYS_SWO: track 0.00 -> 11.2 mm, vias 0 -> 2
- net TIM5_CH2: track 28.8 -> 18.0 mm, vias 2 -> 0
- net /SYS_SWDIO: track 9.72 -> 0.00 mm
- net /SYS_SWO: track 9.18 -> 0.00 mm
- net Net-(SW3A-B): track 0.00 -> 6.36 mm
- net BAT_VSENCE: track 38.4 -> 33.2 mm
- net PYRO_2: track 50.9 -> 55.6 mm
- net GND: track 14.3 -> 10.0 mm, vias 19 -> 21
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- added copper zone on B.Cu, net +5V
- added copper zone on B.Cu, net +BATT
- added copper zone on In1.Cu, net GND
- added copper zone on In2.Cu, net GND
Other:
- copper layers 2 -> 4
- board text added: "ARM"
- board text added: "GND VCC S1 S2"
- board text removed: "GND VCC S2 S1"

Commit message: final touches
Parts:
- moved J1 1.21 mm to (156.2, 103.4)
- moved J12 0.25 mm to (156.2, 116.4)
Routing:
- net +3.3V: track 251.7 -> 254.2 mm
- net +5V: track 74.5 -> 75.3 mm
Other:
- board text added: "VERTEX"
