File: Hardware/flight_comp.kicad_pcb (KiCad board)
At the start: 4 copper layers, 86.7 x 48.2 mm, 127 parts, among them IC1 BMP388, IC4 TPS259531DSGR, J1 Conn_Coaxial, J10 CAMERA_CONN_01, J11 CAMERA_CONN_02, J12 Conn_Coaxial, J13 CAMERA_CONN_03, J2 TC2030, J3 XT30, J4 USB_C_Receptacle_USB2.0_16P, J5 Conn_01x02, J6 Conn_01x02, J7 SERVO_CONN_01, J8 SERVO_CONN_02, J9 SERVO_CONN_02, Q2 DMP3013SFV, Q3 CSD17577Q3A, Q4 CSD17577Q3A, Q5 PMBT2222A, SW1 NRST, SW2 BOOT0, SW3 EG2219, U1 STM32F405RGTx, U10 LTC4412, U11 UCC27517A, U12 UCC27517A, U13 LSM6DSO, U2 MAX-M10S, U3 74LVC1GU04, U4 W25Q32JVSS, U5 24LC64, U6 MP2331, U7 AMS1117-5.0, U8 USBLC6-2SC6, Y1 8mHz, Y2 32.768 kHz

Commit message: Production files
Other:
- board text added: "2S Li-Ion >=20A"
- board text removed: "2-3S Li-Ion >=20A"
Changed lines of the file:
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@@
 			(outputformat 1)
 			(mirror no)
-			(drillshape 1)
+			(drillshape 0)
 			(scaleselection 1)
-			(outputdirectory "")
+			(outputdirectory "C:/Users/kroko/Desktop/Flight_computer/Production/")
 		)
 	)
@@
 			(polygon
 				(pts
-					(xy 143.756958 122.050327) (xy 148.634 123.830858) (xy 148.634 125.240628) (xy 143.756958 127.021158)
-					(xy 143.756958 125.699902) (xy 147.182904 124.51933) (xy 143.756958 123.33905)
+					(xy 143.925779 122.647062) (xy 148.634 124.266978) (xy 148.634 125.466894) (xy 143.925779 127.067173)
+					(xy 143.925779 125.926168) (xy 147.202541 124.945778) (xy 147.462302 124.880644) (xy 147.672073 124.850523)
+					(xy 147.672073 124.830886) (xy 147.448146 124.795455) (xy 147.189352 124.729183) (xy 143.925779 123.75524)
 				)
 			)
 			(polygon
 				(pts
-					(xy 148.634 117.815157) (xy 148.634 121.346615) (xy 143.756958 121.346615) (xy 143.756958 117.815157)
-					(xy 144.694851 117.815157) (xy 144.694851 120.094235) (xy 145.538954 120.094235) (xy 145.538954 117.979288)
-					(xy 146.476847 117.979288) (xy 146.476847 120.094235) (xy 147.696107 120.094235) (xy 147.696107 117.815157)
+					(xy 148.634 119.263907) (xy 148.634 122.08374) (xy 143.925779 122.08374) (xy 143.925779 119.372058)
+					(xy 144.78864 119.372058) (xy 144.78864 121.024801) (xy 145.83908 121.024801) (xy 145.83908 119.48695)
+					(xy 146.701941 119.48695) (xy 146.701941 121.024801) (xy 147.771138 121.024801) (xy 147.771138 119.263907)
 				)
 			)
 			(polygon
 				(pts
-					(xy 148.634 113.596106) (xy 146.852004 114.92762) (xy 146.852004 115.507941) (xy 148.634 115.507941)
-					(xy 148.634 116.760321) (xy 143.756958 116.760321) (xy 143.756958 115.052184) (xy 144.638577 115.052184)
-					(xy 144.638577 115.507941) (xy 145.970385 115.507941) (xy 145.970385 115.12106) (xy 145.962157 114.831645)
-					(xy 145.940489 114.616064) (xy 145.89004 114.42552) (xy 145.804202 114.274905) (xy 145.693272 114.159272)
-					(xy 145.576763 114.083224) (xy 145.440038 114.039416) (xy 145.242932 114.022554) (xy 145.066451 114.042403)
-					(xy 144.924341 114.098171) (xy 144.809045 114.196192) (xy 144.715074 114.356971) (xy 144.673088 114.491451)
-					(xy 144.650301 114.655338) (xy 144.638577 115.052184) (xy 143.756958 115.052184) (xy 143.756958 114.648597)
-					(xy 143.770313 114.230696) (xy 143.806198 113.904438) (xy 143.884058 113.602979) (xy 144.019568 113.3206)
-					(xy 144.208973 113.072472) (xy 144.444551 112.883014) (xy 144.625268 112.795669) (xy 144.840985 112.740351)
-					(xy 145.099317 112.720642) (xy 145.452604 112.751127) (xy 145.742863 112.836437) (xy 145.982401 112.971528)
-					(xy 146.190715 113.155889) (xy 146.37997 113.39209) (xy 146.55012 113.688136) (xy 148.634 112.058255)
+					(xy 148.634 115.782274) (xy 147.423532 116.513538) (xy 147.177628 116.670928) (xy 146.992394 116.823335)
+					(xy 146.874279 116.984242) (xy 146.843646 117.070881) (xy 146.833246 117.166252) (xy 146.833246 117.45143)
+					(xy 148.634 117.45143) (xy 148.634 118.510369) (xy 143.925779 118.510369) (xy 143.925779 116.972519)
+					(xy 144.713609 116.972519) (xy 144.713609 117.45143) (xy 146.045416 117.45143) (xy 146.045416 116.992449)
+					(xy 146.021592 116.773073) (xy 145.954317 116.593382) (xy 145.845235 116.444661) (xy 145.698475 116.327949)
+					(xy 145.532543 116.258621) (xy 145.341117 116.234808) (xy 145.111684 116.265365) (xy 144.944594 116.348914)
+					(xy 144.82358 116.484148) (xy 144.743906 116.683942) (xy 144.713609 116.972519) (xy 143.925779 116.972519)
+					(xy 143.925779 116.831542) (xy 143.952504 116.372858) (xy 144.025235 116.010675) (xy 144.135193 115.727364)
+					(xy 144.277242 115.508166) (xy 144.450364 115.341925) (xy 144.657791 115.221944) (xy 144.906641 115.146672)
+					(xy 145.207175 115.119888) (xy 145.446883 115.139276) (xy 145.662053 115.195505) (xy 145.86098 115.286723)
+					(xy 146.038382 115.408583) (xy 146.193268 115.559503) (xy 146.32737 115.741535) (xy 146.43487 115.945431)
+					(xy 146.517879 116.175896) (xy 146.531069 116.175896) (xy 146.573426 116.074043) (xy 146.637754 115.972784)
+					(xy 146.809799 115.782568) (xy 147.021411 115.607006) (xy 147.242988 115.454598) (xy 148.634 114.565945)
 				)
 			)
 			(polygon
 				(pts
-					(xy 144.694851 107.688262) (xy 144.694851 109.212923) (xy 148.634 109.212923) (xy 148.634 110.472044)
-					(xy 144.694851 110.472044) (xy 144.694851 111.996706) (xy 143.756958 111.996706) (xy 143.756958 107.688262)
+					(xy 144.78864 110.997264) (xy 144.78864 112.33845) (xy 148.634 112.33845) (xy 148.634 113.400907)
+					(xy 144.78864 113.400907) (xy 144.78864 114.735352) (xy 143.925779 114.735352) (xy 143.925779 110.997264)
 				)
 			)
 			(polygon
 				(pts
-					(xy 148.634 103.399748) (xy 148.634 106.931207) (xy 143.756958 106.931207) (xy 143.756958 103.399748)
-					(xy 144.694851 103.399748) (xy 144.694851 105.678827) (xy 145.538954 105.678827) (xy 145.538954 103.563879)
-					(xy 146.476847 103.563879) (xy 146.476847 105.678827) (xy 147.696107 105.678827) (xy 147.696107 103.399748)
+					(xy 148.634 107.54494) (xy 148.634 110.364773) (xy 143.925779 110.364773) (xy 143.925779 107.653091)
+					(xy 144.78864 107.653091) (xy 144.78864 109.305833) (xy 145.83908 109.305833) (xy 145.83908 107.767983)
+					(xy 146.701941 107.767983) (xy 146.701941 109.305833) (xy 147.771138 109.305833) (xy 147.771138 107.54494)
 				)
 			)
 			(polygon
 				(pts
-					(xy 148.634 97.918353) (xy 148.634 99.374138) (xy 147.029031 100.426629) (xy 148.634 101.49905)
-					(xy 148.634 102.889183) (xy 146.1776 101.157892) (xy 143.756958 102.853133) (xy 143.756958 101.400572)
-					(xy 145.276637 100.384131) (xy 143.756958 99.338087) (xy 143.756958 97.944731) (xy 146.128361 99.649644)
+					(xy 148.634 102.923768) (xy 148.634 104.179371) (xy 147.100838 104.989476) (xy 146.996266 105.030817)
+					(xy 146.785472 105.084438) (xy 146.785472 105.097627) (xy 147.113734 105.205778) (xy 148.634 106.019106)
+					(xy 148.634 107.281451) (xy 146.279889 105.782875) (xy 143.925779 107.153663) (xy 143.925779 105.86494)
+					(xy 145.3376 105.192882) (xy 145.513952 105.120574) (xy 145.734739 105.051905) (xy 145.734739 105.038715)
+					(xy 145.324411 104.89129) (xy 143.925779 104.143614) (xy 143.925779 102.963042) (xy 146.260252 104.373105)
 				)
 			)
@@
 		)
 	)
-	(gr_text "2-3S\nLi-Ion\n>=20A"
+	(gr_text "2S\nLi-Ion\n>=20A"
 		(at 90.45 112.1 0)
 		(layer "F.SilkS" knockout)
