File: Hardware/sensors.kicad_sch (KiCad schematic)
At the start: 29 parts, among them IC1 BMP388, J1 Conn_Coaxial, J12 Conn_Coaxial, U13 LSM6DSO, U2 MAX-M10S, U3 74LVC1GU04

Commit message: PCB added, minor changes
Parts:
- IC1: footprint BMP388 -> Package_LGA:ST_HLGA-10_2x2mm_P0.5mm_LayoutBorder3x2y
- R24, R25, R26, R27: footprint (none) -> Resistor_SMD:R_0603_1608Metric
- U13: footprint LSM6DSO:LGA14L -> Package_LGA:LGA-14_3x2.5mm_P0.5mm_LayoutBorder3x4y
- U2: footprint MAX-M10S:MAXM10M00B -> RF_GPS:ublox_MAX
- U3: footprint (none) -> Package_TO_SOT_SMD:SOT-23-5

Commit message: Kaut ko palaboju
Other:
- note added: "BARO"
- note removed: "BMP388"
- moved on the sheet: C1, C2, C3, C4, C41, C42, C5, D5, E22-400M22S2, IC1, J1, J12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
